File: Hardware_design/Buttons_circuits.kicad_sch (KiCad schematic)
At the start: 63 parts

Commit message: Buttons number modified
now the buttons are 10, one is for starting and stoping the count and another one for reseting it
Parts:
- removed C? (x5): 0.1 uF, symbol Device:C
- removed R? (x5): 220, symbol Device:R
- removed R? (x5): 10k, symbol Device:R
- removed SW? (x5): ADTS24NV, ADTS24*V_APM, symbol PUSH_BUTTON_ADTS24NV:ADTS24NV
- removed U?: 74HC14D_653, 74HC14D_653:SOIC127P600X175-14N, symbol Schimitt_Trigger_74HC14D_653:74HC14D_653
Connections:
- net PAUSE_1 is gone; now on net RESET_1: U?.3 (2A)
- net PAUSE_1_FILTERED is gone; now on net RESET_1_FILTERED: U?.4 (2Y)
- net PAUSE_3 is gone; now on net RESET_4: U?.3 (2A)
- net PAUSE_3_FILTERED is gone; now on net RESET_4_FILTERED: U?.4 (2Y)
- net START_2_FILTERED is gone; now on net RESET_2_FILTERED: U?.8 (4Y)
- net START_4_FILTERED is gone; now on net RESET_5_FILTERED: U?.8 (4Y)
- net RESET_1: no longer U?.5 (3A)
- net RESET_1_FILTERED: no longer U?.6 (3Y)
- net RESET_2: now also U?.9 (4A); no longer U?.13 (6A)
- net RESET_2_FILTERED: no longer U?.12 (6Y)
- net RESET_3: now also U?.13 (6A); no longer U?.5 (3A)
- net RESET_3_FILTERED: now also U?.12 (6Y); no longer U?.6 (3Y)
- net RESET_4: no longer U?.13 (6A)
- net RESET_4_FILTERED: no longer U?.12 (6Y)
- net RESET_5: now also U?.9 (4A)
- net PAUSE_2 renamed START_STOP_3
- net START_STOP_3: now also C?.1, R?.2
- net PAUSE_2_FILTERED renamed START_STOP_3_FILTERED
- net PAUSE_4: no longer names the net of U?.11 (5A)
- net PAUSE_4_FILTERED: no longer names the net of U?.10 (5Y)
- net START_1 renamed START_STOP_1
- net START_1_FILTERED renamed START_STOP_1_FILTERED
- net START_2 renamed START_STOP_2
- net START_STOP_2: now also U?.5 (3A); no longer U?.9 (4A)
- removed net START_3: C?.1, R?.2, U?.1 (1A)
- net START_3_FILTERED renamed START_STOP_4_FILTERED
- net START_4 renamed START_STOP_4
- net START_STOP_4: now also U?.1 (1A); no longer U?.9 (4A)
- net START_5 renamed START_STOP_5
- net START_STOP_5: now also U?.5 (3A)
- new net START_STOP_2_FILTERED: U?.6 (3Y)
- new net START_STOP_5_FILTERED: U?.6 (3Y)
- no-connect marks 6 -> 4
Other:
- moved on the sheet: C?, R?, SW?, U?

Commit message: starting footprint asignment
Parts:
- C25, C26, C27, C28, C29, C30, C31, C32, C33, C34: renamed from C?; footprint (none) -> Footprints:0805_SMD_CERAMIC_CAP_T491B106K016AT
- SW10, SW11, SW12, SW3, SW4, SW5, SW6, SW7, SW8, SW9: renamed from SW?; footprint ADTS24*V_APM -> Footprints:PUSH_BUTTON_ADTS24NV
- U15, U16: renamed from U?; footprint 74HC14D_653:SOIC127P600X175-14N -> Footprints:Schimitt_Trigger_74HC14D_653
- gave numbers to parts that had none: 20

Commit message: all footprints asigned
Parts:
- R23, R24, R25, R26, R27, R28, R29, R30, R31, R32, R33, R34, R35, R36, R37, R38, R39, R40, R41, R42: footprint (none) -> Footprints:0805_RES_RESC2012X60N
Changed lines of the file:
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@@
 			)
 		)
-		(property "Footprint" ""
+		(property "Footprint" "Footprints:0805_RES_RESC2012X60N"
 			(at 90.17 411.988 90)
 			(hide yes)
@@
 			)
 		)
-		(property "Footprint" ""
+		(property "Footprint" "Footprints:0805_RES_RESC2012X60N"
 			(at 40.132 111.76 90)
 			(hide yes)
@@
 			)
 		)
-		(property "Footprint" ""
+		(property "Footprint" "Footprints:0805_RES_RESC2012X60N"
 			(at 79.502 111.76 90)
 			(hide yes)
@@
 			)
 		)
-		(property "Footprint" ""
+		(property "Footprint" "Footprints:0805_RES_RESC2012X60N"
 			(at 40.132 288.29 90)
 			(hide yes)
@@
 			)
 		)
-		(property "Footprint" ""
+		(property "Footprint" "Footprints:0805_RES_RESC2012X60N"
 			(at 50.8 104.648 90)
 			(hide yes)
@@
 			)
 		)
-		(property "Footprint" ""
+		(property "Footprint" "Footprints:0805_RES_RESC2012X60N"
 			(at 40.132 199.39 90)
 			(hide yes)
@@
 			)
 		)
-		(property "Footprint" ""
+		(property "Footprint" "Footprints:0805_RES_RESC2012X60N"
 			(at 79.502 419.1 90)
 			(hide yes)
@@
 			)
 		)
-		(property "Footprint" ""
+		(property "Footprint" "Footprints:0805_RES_RESC2012X60N"
 			(at 90.17 192.278 90)
 			(hide yes)
@@
 			)
 		)
-		(property "Footprint" ""
+		(property "Footprint" "Footprints:0805_RES_RESC2012X60N"
 			(at 50.8 192.278 90)
 			(hide yes)
@@
 			)
 		)
-		(property "Footprint" ""
+		(property "Footprint" "Footprints:0805_RES_RESC2012X60N"
 			(at 79.502 506.73 90)
 			(hide yes)
@@
 			)
 		)
-		(property "Footprint" ""
+		(property "Footprint" "Footprints:0805_RES_RESC2012X60N"
 			(at 40.132 419.1 90)
 			(hide yes)
@@
 			)
 		)
-		(property "Footprint" ""
+		(property "Footprint" "Footprints:0805_RES_RESC2012X60N"
 			(at 50.8 411.988 90)
 			(hide yes)
@@
 			)
 		)
-		(property "Footprint" ""
+		(property "Footprint" "Footprints:0805_RES_RESC2012X60N"
 			(at 50.8 499.618 90)
 			(hide yes)
@@
 			)
 		)
-		(property "Footprint" ""
+		(property "Footprint" "Footprints:0805_RES_RESC2012X60N"
 			(at 79.502 288.29 90)
 			(hide yes)
@@
 			)
 		)
-		(property "Footprint" ""
+		(property "Footprint" "Footprints:0805_RES_RESC2012X60N"
 			(at 79.502 199.39 90)
 			(hide yes)
@@
 			)
 		)
-		(property "Footprint" ""
+		(property "Footprint" "Footprints:0805_RES_RESC2012X60N"
 			(at 40.132 506.73 90)
 			(hide yes)
@@
 			)
 		)
-		(property "Footprint" ""
+		(property "Footprint" "Footprints:0805_RES_RESC2012X60N"
 			(at 90.17 499.618 90)
 			(hide yes)
@@
 			)
 		)
-		(property "Footprint" ""
+		(property "Footprint" "Footprints:0805_RES_RESC2012X60N"
 			(at 90.17 281.178 90)
 			(hide yes)
@@
 			)
 		)
-		(property "Footprint" ""
+		(property "Footprint" "Footprints:0805_RES_RESC2012X60N"
 			(at 50.8 281.178 90)
 			(hide yes)
@@
 			)
 		)
-		(property "Footprint" ""
+		(property "Footprint" "Footprints:0805_RES_RESC2012X60N"
 			(at 90.17 104.648 90)
 			(hide yes)

Commit message: Index problem solved and some progress made
Parts:
- added D10, D11, D12, D3, D4, D5, D6, D7, D8, D9: D_Schottky, Footprints:DIO_Schottky _MBR0530T3G, symbol Device:D_Schottky
Connections:
- net RESET_1_FILTERED: now also D4.1 (K)
- net RESET_2_FILTERED: now also D6.1 (K)
- net RESET_3_FILTERED: now also D8.1 (K)
- net RESET_4_FILTERED: now also D10.1 (K)
- net RESET_5_FILTERED: now also D12.1 (K)
- net START_STOP_1_FILTERED: now also D3.C (K)
- net START_STOP_2_FILTERED: now also D5.1 (K)
- net START_STOP_3_FILTERED: now also D7.1 (K)
- net START_STOP_4_FILTERED: now also D9.1 (K)
- net START_STOP_5_FILTERED: now also D11.1 (K)
- new net DIO_INDEX: D10.2 (A), D11.2 (A), D12.2 (A), D3.A, D4.2 (A), D5.2 (A), D6.2 (A), D7.2 (A), D8.2 (A), D9.2 (A)

Commit message: big update
coper zones already set, edgecuts set, all components placed, we are just missing the routing
Parts:
- removed C34: 0.1 uF, Footprints:0805_SMD_CERAMIC_CAP_T491B106K016AT, symbol Device:C
- removed D11, D12: D_Schottky, Footprints:DIO_Schottky _MBR0530T3G, symbol Device:D_Schottky
- removed R37: 10k, Footprints:0805_RES_RESC2012X60N, symbol Device:R
- removed R42: 220, Footprints:0805_RES_RESC2012X60N, symbol Device:R
- removed SW12: ADTS24NV, Footprints:PUSH_BUTTON_ADTS24NV, symbol PUSH_BUTTON_ADTS24NV:ADTS24NV
Connections:
- net DIO_INDEX: now also D10.A, D4.A, D5.A, D6.A, D7.A, D8.A, D9.A; no longer D10.2 (A), D4.2 (A), D5.2 (A), D6.2 (A), D7.2 (A), D8.2 (A), D9.2 (A)
- net RESET_1_FILTERED: now also D4.C (K); no longer D4.1 (K)
- net RESET_2_FILTERED: now also D6.C (K); no longer D6.1 (K)
- net RESET_3_FILTERED: now also D8.C (K); no longer D8.1 (K)
- net RESET_4_FILTERED: now also D10.C (K); no longer D10.1 (K)
- net START_STOP_2_FILTERED: now also D5.C (K); no longer D5.1 (K)
- net START_STOP_3_FILTERED: now also D7.C (K); no longer D7.1 (K)
- net START_STOP_4_FILTERED: now also D9.C (K); no longer D9.1 (K)
- net RESET_5: no longer names the net of U15.9 (4A)
- net RESET_5_FILTERED: no longer names the net of U15.8 (4Y)
- net START_STOP_5 renamed ALARM_OFF
- net START_STOP_5_FILTERED renamed ALARM_OFF_FILTERED
- no-connect marks 4 -> 6

Commit message: a little advance
Parts:
- added C23, C24: 10uF, Footprints:0805_SMD_TANT_CAP_T491B106K016AT, symbol Device:C
Connections:
- net +3.3V: now also C23.1, C24.1
- net GND: now also C23.2, C24.2
