File: Hardware_design/Hardware_design.kicad_pcb (KiCad board)
At the start: 2 copper layers, 227 parts, among them IC1 ESP32-S3-WROOM-1-N16, J1 FTSH-103-01-F-D, J2 SBH11-PBPC-D05-ST-BK, J3 54-00131, SW1 TL3301FF160QG, SW10 ADTS24NV, SW11 ADTS24NV, SW12 ADTS24NV, SW2 TL3301FF160QG, SW3 ADTS24NV, SW4 ADTS24NV, SW5 ADTS24NV, SW6 ADTS24NV, SW7 ADTS24NV, SW8 ADTS24NV, SW9 ADTS24NV, U1 LS7366R-S, U10 MAX7221CWG_, U11 MAX7221CWG_, U12 MAX7221CWG_, U13 MAX7221CWG_, U14 MAX7221CWG_, U15 74HC14D_653, U16 74HC14D_653, U2 TXB0104DR, U3 LP3875EMP-3.3, U4 MAX7221CWG_, U5 MAX7221CWG_, U6 MAX7221CWG_, U7 MAX7221CWG_, U8 MAX7221CWG_, U9 MAX7221CWG_

Commit message: pcb layout started
concecting first MAX7221 and its 8 displays
Parts:
- moved DS13 433.3 mm to (247.7, 73.5)
- moved DS14 433.3 mm to (258.1, 73.5)
- moved DS15 433.3 mm to (268.5, 73.5)
- moved DS56 432.9 mm to (237.3, 73.5)
- moved DS45 414.9 mm to (216.5, 31.5)
- moved DS46 414.9 mm to (226.9, 31.5)
- moved DS47 414.9 mm to (237.3, 31.5)
- moved DS48 414.9 mm to (247.7, 31.5)
- moved DS5 411.1 mm to (258.1, 31.5)
- moved DS6 411.1 mm to (268.5, 31.5)
- moved DS49 402.1 mm to (247.7, 52.5)
- moved DS7 402.0 mm to (268.5, 52.5)
- moved DS12 391.9 mm to (195.7, 73.5)
- moved DS50 381.4 mm to (237.3, 52.5)
- moved DS8 381.3 mm to (258.1, 52.5)
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Routing:
- net /Display_management/SEG_D_MAX7221_1: track 0.00 -> 122.3 mm, vias 0 -> 2
- net /Display_management/SEG_F_MAX7221_1: track 0.00 -> 121.8 mm
- net /Display_management/SEG_DP_MAX7221_1: track 0.00 -> 121.3 mm, vias 0 -> 2
- net /Display_management/SEG_B_MAX7221_1: track 0.00 -> 119.2 mm, vias 0 -> 2
- net /Display_management/SEG_E_MAX7221_1: track 0.00 -> 112.8 mm, vias 0 -> 9
- net /Display_management/SEG_A_MAX7221_1: track 0.00 -> 112.1 mm, vias 0 -> 8
- net /Display_management/SEG_C_MAX7221_1: track 0.00 -> 110.7 mm, vias 0 -> 9
- net /Display_management/SEG_G_MAX7221_1: track 0.00 -> 109.7 mm, vias 0 -> 8
- net /Display_management/DIG_6_MAX7221_1: track 0.00 -> 91.3 mm, vias 0 -> 2
- net /Display_management/DIG_4_MAX7221_1: track 0.00 -> 70.3 mm, vias 0 -> 2
- net /Display_management/DIG_2_MAX7221_1: track 0.00 -> 47.4 mm, vias 0 -> 2
- net /Display_management/DIG_0_MAX7221_1: track 0.00 -> 26.3 mm, vias 0 -> 2
- net Net-(U4-DOUT): track 0.00 -> 25.9 mm
- net /SCK_MAX7221_5V: track 0.00 -> 23.5 mm
- net /Display_management/DIG_1_MAX7221_1: track 0.00 -> 3.50 mm, vias 0 -> 1

Commit message: 10 uF display caps deleted
10 uF display caps ocupy too much space, they were deleted
Parts:
- removed C39, C40, C41, C42, C43, C44, C45, C46, C47, C48: 10uF, Footprints:0805_SMD_TANT_CAP_T491B106K016AT
- moved U12 259.3 mm to (164.1, 144.5)
- moved U13 254.3 mm to (164.0, 163.9)
- moved U14 251.8 mm to (163.6, 184.2)
- moved C38 241.7 mm to (159.6, 30.8), turned to -90 degrees
- moved C14 225.5 mm to (156.5, 30.8), turned to -90 degrees
- moved R12 201.1 mm to (141.1, 30.2)
- moved TP17 6.40 mm to (-40.3, 74.9)
- moved DS10 4.00 mm to (174.7, 77.5)
- moved DS11 4.00 mm to (185.1, 77.5)
- moved DS12 4.00 mm to (195.7, 77.5)
- moved DS13 4.00 mm to (247.7, 77.5)
- moved DS14 4.00 mm to (258.1, 77.5)
- moved DS15 4.00 mm to (268.5, 77.5)
- moved DS53 4.00 mm to (206.3, 77.5)
- moved DS54 4.00 mm to (216.5, 77.5)
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Routing:
- net /Display_management/DIG_6_MAX7221_1: track 91.3 -> 0.00 mm, vias 2 -> 0
- net /Display_management/DIG_4_MAX7221_1: track 70.3 -> 0.00 mm, vias 2 -> 0
- net /Display_management/DIG_2_MAX7221_1: track 47.4 -> 0.00 mm, vias 2 -> 0
- net /Display_management/DIG_0_MAX7221_1: track 26.3 -> 0.00 mm, vias 2 -> 0
- net Net-(U4-DOUT): track 25.9 -> 0.00 mm
- net /SCK_MAX7221_5V: track 23.5 -> 0.00 mm
- net /Display_management/SEG_DP_MAX7221_1: track 121.3 -> 100.7 mm, vias 2 -> 0
- net /Display_management/SEG_B_MAX7221_1: track 119.2 -> 101.1 mm, vias 2 -> 0
- net /Display_management/SEG_D_MAX7221_1: track 122.3 -> 104.6 mm, vias 2 -> 0
- net /Display_management/SEG_A_MAX7221_1: track 112.1 -> 94.7 mm
- net /Display_management/SEG_E_MAX7221_1: track 112.8 -> 96.4 mm, vias 9 -> 8
- net /Display_management/SEG_C_MAX7221_1: track 110.7 -> 94.7 mm, vias 9 -> 8
- net /Display_management/SEG_G_MAX7221_1: track 109.7 -> 95.1 mm
- net /Display_management/SEG_F_MAX7221_1: track 121.8 -> 107.5 mm
- net /Display_management/DIG_1_MAX7221_1: track 3.50 -> 0.00 mm, vias 1 -> 0

Commit message: component placement started
index pin and gpio pins for 10 buttons problem, index pin should be activated whenever any of the 10 buttons is pressed but only the gpio pin of the button that was pressed should also be activaded
Parts:
- removed C38: 10uF, Footprints:0805_SMD_TANT_CAP_T491B106K016AT
- C14: moved to B.Cu
- moved U16 503.1 mm to (336.5, 64.6)
- moved SW10 487.8 mm to (303.1, 122.2)
- moved C32 487.8 mm to (324.5, 122.7)
- moved R35 487.8 mm to (328.2, 97.9)
- moved R40 487.8 mm to (332.6, 97.9)
- moved C28 463.4 mm to (299.0, 168.1)
- moved C29 463.4 mm to (299.0, 171.1)
- moved C33 463.4 mm to (303.8, 168.1)
- moved C34 463.4 mm to (303.8, 171.1)
- moved R26 463.4 mm to (298.8, 143.3)
- moved R27 463.4 mm to (298.8, 146.2)
- moved R31 463.4 mm to (303.1, 143.3)
- moved R32 463.4 mm to (303.1, 146.2)
- moved R36 463.4 mm to (307.5, 143.3)
- moved R37 463.4 mm to (307.5, 146.2)
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Routing:
- net /Display_management/DIG_7_MAX7221_1: track 0.00 -> 105.1 mm, vias 0 -> 4
- net /Display_management/DIG_6_MAX7221_1: track 0.00 -> 94.7 mm, vias 0 -> 2
- net /Display_management/DIG_5_MAX7221_1: track 0.00 -> 82.0 mm, vias 0 -> 4
- net /Display_management/DIG_4_MAX7221_1: track 0.00 -> 72.7 mm, vias 0 -> 2
- net /Display_management/DIG_3_MAX7221_1: track 0.00 -> 64.0 mm, vias 0 -> 2
- net /Display_management/DIG_2_MAX7221_1: track 0.00 -> 55.0 mm, vias 0 -> 2
- net /Display_management/DIG_1_MAX7221_1: track 0.00 -> 39.2 mm, vias 0 -> 2
- net /LFLAG: track 0.00 -> 33.9 mm, vias 0 -> 2
- net /ESP_TMS: track 0.00 -> 32.8 mm, vias 0 -> 2
- net /ESP_IO0: track 0.00 -> 32.2 mm, vias 0 -> 2
- net /Display_management/SEG_C_MAX7221_1: track 94.7 -> 125.6 mm, vias 8 -> 9
- net /Display_management/SEG_B_MAX7221_1: track 101.1 -> 131.8 mm, vias 0 -> 3
- net /Display_management/DIG_0_MAX7221_1: track 0.00 -> 28.7 mm
- net /Display_management/SEG_DP_MAX7221_1: track 100.7 -> 129.2 mm, vias 0 -> 2
- net /Display_management/SEG_F_MAX7221_1: track 107.5 -> 136.0 mm, vias 0 -> 2
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
Commit message: Index problem solved and some progress made
Parts:
- added D10: D_Schottky, Footprints:DIO_Schottky _MBR0530T3G, F.Cu at (265.2, 137.0)
- added D11: D_Schottky, Footprints:DIO_Schottky _MBR0530T3G, F.Cu at (265.2, 140.1)
- added D12: D_Schottky, Footprints:DIO_Schottky _MBR0530T3G, F.Cu at (265.2, 143.3)
- added D3: D_Schottky, Footprints:DIO_Schottky _MBR0530T3G, F.Cu at (235.0, 59.5)
- added D4: D_Schottky, Footprints:DIO_Schottky _MBR0530T3G, F.Cu at (235.0, 62.6)
- added D5: D_Schottky, Footprints:DIO_Schottky _MBR0530T3G, F.Cu at (235.0, 65.8)
- added D6: D_Schottky, Footprints:DIO_Schottky _MBR0530T3G, F.Cu at (235.0, 69.0)
- added D7: D_Schottky, Footprints:DIO_Schottky _MBR0530T3G, F.Cu at (235.0, 72.2)
- added D8: D_Schottky, Footprints:DIO_Schottky _MBR0530T3G, F.Cu at (235.0, 75.4)
- added D9: D_Schottky, Footprints:DIO_Schottky _MBR0530T3G, F.Cu at (265.2, 133.8)
- moved DS67 409.8 mm to (214.8, 101.9)
- moved DS68 401.4 mm to (214.8, 78.9)
- moved DS23 379.5 mm to (173.2, 147.9)
- moved DS24 379.5 mm to (183.6, 147.9)
- moved DS57 377.9 mm to (194.0, 101.9)
- moved DS58 377.9 mm to (204.4, 101.9)
- moved DS78 374.7 mm to (173.2, 216.9)
- moved DS79 374.7 mm to (183.6, 216.9)
- moved DS80 374.7 mm to (194.0, 216.9)
- moved DS60 371.1 mm to (214.8, 55.9)
- moved DS81 369.8 mm to (194.0, 239.9)
- moved DS59 368.6 mm to (204.4, 78.9)
- moved DS41 366.9 mm to (204.4, 239.9)
- moved DS42 366.9 mm to (214.8, 239.9)
- moved DS82 364.5 mm to (204.4, 216.9)
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Routing:
- net /RESET_3_FILTERED: track 0.00 -> 16.4 mm, vias 0 -> 2
- net /INDEX: track 11.3 -> 27.2 mm
- net /Buttons_circuits/RESET_3: track 0.00 -> 15.5 mm, vias 0 -> 2
- net unconnected-(U15-6A-Pad13): track 0.00 -> 15.5 mm, vias 0 -> 2
- net /START_STOP_5_FILTERED: track 0.00 -> 14.6 mm
- net /RESET_2_FILTERED: track 0.00 -> 13.5 mm
- net /START_STOP_3_FILTERED: track 0.00 -> 13.0 mm, vias 0 -> 2
- net unconnected-(U15-6Y-Pad12): track 0.00 -> 12.7 mm, vias 0 -> 2
- net unconnected-(U15-5Y-Pad10): track 0.00 -> 12.6 mm, vias 0 -> 2
- net /Buttons_circuits/START_STOP_5: track 0.00 -> 11.9 mm, vias 0 -> 2
- net /Buttons_circuits/START_STOP_2: track 0.00 -> 11.9 mm, vias 0 -> 2
- net /Buttons_circuits/START_STOP_4: track 0.00 -> 11.6 mm
- net /Buttons_circuits/START_STOP_1: track 0.00 -> 11.6 mm
- net /Buttons_circuits/RESET_4: track 0.00 -> 11.0 mm, vias 0 -> 2
- net /Buttons_circuits/RESET_1: track 0.00 -> 11.0 mm, vias 0 -> 2
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
Commit message: big update
coper zones already set, edgecuts set, all components placed, we are just missing the routing
Parts:
- removed C23, C24, C34: 0.1 uF, Footprints:0805_SMD_CERAMIC_CAP_T491B106K016AT
- removed D11, D12: D_Schottky, Footprints:DIO_Schottky _MBR0530T3G
- removed DS37, DS38, DS39, DS40, DS41, DS42, DS43, DS44, DS77, DS78, DS79, DS80, DS81, DS82, DS83, DS84, DS85: ACSC03-41EWA-F01, Footprints:SMD_DISPLAY_ACSC03-41EWA-F01
- removed R37: 10k, Footprints:0805_RES_RESC2012X60N
- removed R42: 220, Footprints:0805_RES_RESC2012X60N
- removed SW12: ADTS24NV, Footprints:PUSH_BUTTON_ADTS24NV
- removed TP10, TP11, TP12, TP13, TP14, TP16, TP17, TP9: TestPoint, TestPoint:TestPoint_Pad_1.0x1.0mm
- removed U13, U14: MAX7221CWG_, Footprints:Disp_Controler_MAX7221CWG_
- added LS1: CMI-9605IC-0580T, Footprints:BUZZER_CMI-9605IC-0580T, F.Cu at (88.5, 101.8)
- added Q1: MMBT2222A, Footprints:TRANSISTOR_MMBT2222A, F.Cu at (85.2, 94.6)
- C14: moved to F.Cu
- R21: value 3v=24.5k, 1.8v=29.8k -> 1k
- R22: value 3v=24.5k, 1.8v=29.8k -> 10k
- moved C22 409.1 mm to (237.6, 159.4), turned to -90 degrees
- moved R20 405.6 mm to (242.9, 159.4), turned to -90 degrees
- moved TP15 384.9 mm to (230.9, 149.2)
- moved C21 288.9 mm to (106.8, 194.2), turned to -90 degrees
- moved R19 285.4 mm to (112.0, 194.3), turned to -90 degrees
- moved C15 284.5 mm to (106.5, 56.1), turned to -90 degrees
- moved C19 281.6 mm to (106.8, 147.9), turned to -90 degrees
- moved TP8 280.8 mm to (100.2, 46.0)
- moved R13 280.7 mm to (112.1, 56.3), turned to -90 degrees
- moved C17 280.1 mm to (106.5, 102.4), turned to -90 degrees
- moved C20 280.1 mm to (103.4, 171.1), turned to -90 degrees
- moved C16 278.0 mm to (103.0, 79.4), turned to -90 degrees
- moved R17 277.7 mm to (112.1, 148.3), turned to -90 degrees
- moved C18 277.1 mm to (103.5, 125.3), turned to -90 degrees
- moved R18 276.5 mm to (108.6, 171.3), turned to -90 degrees
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Connections:
- net /Buttons_circuits/START_STOP_5 renamed /Buttons_circuits/ALARM_OFF
- IC1 pad 24: /START_STOP_5_FILTERED -> /Alarm_OFF_FILTERED
- IC1 pad 25: /RESET_5_FILTERED -> /BUZZER_GPIO_OUT
- R21 pad 1: +5V -> /BUZZER_GPIO_OUT
- R21 pad 2: Net-(U13-ISET) -> Net-(Q1-Pad1)
- R22 pad 1: +5V -> Net-(Q1-Pad1)
- R22 pad 2: Net-(U14-ISET) -> GND
- U12 pad 10: /Display_management/DIG_5_MAX7221_9 -> unconnected-(U12-DIG_5-Pad10)
- U12 pad 24: Net-(U12-DOUT) -> unconnected-(U12-DOUT-Pad24)
- U12 pad 3: /Display_management/DIG_4_MAX7221_9 -> unconnected-(U12-DIG_4-Pad3)
- U12 pad 5: /Display_management/DIG_6_MAX7221_9 -> unconnected-(U12-DIG_6-Pad5)
- U12 pad 8: /Display_management/DIG_7_MAX7221_9 -> unconnected-(U12-DIG_7-Pad8)
- U15 pad 6: /RESET_5_FILTERED -> /Alarm_OFF_FILTERED
- U15 pad 8: /START_STOP_5_FILTERED -> unconnected-(U15-4Y-Pad8)
- U15 pad 9: /Buttons_circuits/RESET_5 -> unconnected-(U15-4A-Pad9)
Routing:
- net /START_STOP_1_FILTERED: track 9.15 -> 533.8 mm, vias 0 -> 2
- net /START_STOP_3_FILTERED: track 13.0 -> 537.2 mm, vias 2 -> 4
- net /RESET_2_FILTERED: track 13.5 -> 537.3 mm, vias 0 -> 2
- net /RESET_1_FILTERED: track 8.30 -> 532.0 mm, vias 0 -> 2
- net /START_STOP_2_FILTERED: track 7.92 -> 531.2 mm, vias 0 -> 2
- net /RESET_3_FILTERED: track 16.4 -> 536.3 mm, vias 2 -> 4
- net /Buttons_circuits/RESET_4: track 11.0 -> 330.4 mm, vias 2 -> 0
- net /Display_management/SEG_F_MAX7221_2: track 0.00 -> 187.4 mm, vias 0 -> 4
- net /Display_management/SEG_D_MAX7221_2: track 0.00 -> 183.7 mm, vias 0 -> 2
- net /Display_management/SEG_A_MAX7221_2: track 0.00 -> 182.6 mm, vias 0 -> 14
- net /Display_management/SEG_B_MAX7221_2: track 0.00 -> 178.9 mm, vias 0 -> 4
- net /Display_management/SEG_C_MAX7221_2: track 0.00 -> 174.2 mm, vias 0 -> 12
- net /Display_management/SEG_DP_MAX7221_2: track 0.00 -> 167.2 mm, vias 0 -> 4
- net /Display_management/SEG_G_MAX7221_2: track 0.00 -> 162.6 mm, vias 0 -> 14
- net /Display_management/SEG_E_MAX7221_2: track 0.00 -> 160.6 mm, vias 0 -> 12
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- added copper zone on B.Cu, net +3.3V
- added copper zone on F.Cu, net +3.3V
- added copper zone on F.Cu, net +5V
- added copper zone on B.Cu, net GND
- added copper zone on F.Cu, net GND
Other:
- board outline added: 231.3 x 191.9 mm

Commit message: a little advance
Parts:
- added C23: 10uF, Footprints:0805_SMD_TANT_CAP_T491B106K016AT, F.Cu at (78.8, 81.1)
- added C24: 10uF, Footprints:0805_SMD_TANT_CAP_T491B106K016AT, F.Cu at (255.0, 104.7)
- moved R21 14.3 mm to (85.0, 86.9)
- moved C13 13.0 mm to (77.2, 56.4), turned to -90 degrees
- moved D10 11.9 mm to (68.1, 83.7)
- moved R22 9.88 mm to (85.0, 89.4)
- moved R9 8.62 mm to (92.8, 56.3), turned to 180 degrees
- moved TP2 8.33 mm to (74.0, 50.9)
- moved Q1 7.37 mm to (89.0, 88.2)
- moved D9 7.03 mm to (70.7, 83.7)
- moved LS1 5.63 mm to (89.9, 96.4), turned to 0 degrees
- moved D2 3.35 mm to (92.9, 53.8), turned to 180 degrees
- moved C11 2.16 mm to (44.5, 37.5)
- moved R10 2.00 mm to (44.7, 35.2)
- moved J1 0.93 mm to (78.8, 32.1)
- moved C4 0.78 mm to (51.3, 32.6)
- moved TP3 0.72 mm to (89.9, 69.3)
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Routing:
- net /INDEX: track 11.3 -> 423.5 mm, vias 0 -> 4
- net /Buttons_circuits/START_STOP_4: track 0.00 -> 320.1 mm, vias 0 -> 4
- net GND: track 5.88 -> 107.7 mm, vias 0 -> 24
- net +3.3V: track 6.92 -> 87.2 mm, vias 0 -> 3
- net /RESET_4_FILTERED: track 0.00 -> 48.0 mm, vias 0 -> 2
- net /OE: track 0.00 -> 45.9 mm, vias 0 -> 2
- net /START_STOP_4_FILTERED: track 0.00 -> 43.3 mm, vias 0 -> 2
- net /Pulse_Signal: track 0.00 -> 40.1 mm
- net /SCK_MAX7221: track 0.00 -> 31.7 mm, vias 0 -> 2
- net /MOSI_MAX7221: track 0.00 -> 31.3 mm, vias 0 -> 2
- net /CS_MAX7221: track 0.00 -> 30.8 mm, vias 0 -> 2
- net Net-(R27-Pad1): track 0.00 -> 28.5 mm, vias 0 -> 1
- net /ESP_EN: track 26.0 -> 51.9 mm, vias 0 -> 4
- net Net-(R26-Pad1): track 0.00 -> 25.4 mm
- net /MOSI_MAX7221_5V: track 0.00 -> 22.5 mm, vias 0 -> 2
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Other:
- outline, holes or cut-outs redrawn

Commit message: update
Parts:
- J2: value SBH11-PBPC-D05-ST-BK -> Conn_01x04_Pin; footprint Footprints:JTAG_2.54_SBH11-PBPC-D05-ST-BK -> Footprints:Jtag_pins
- moved J2 29.6 mm to (74.5, 51.6), turned to 0 degrees
- moved TP2 8.76 mm to (81.5, 55.4)
- moved D2 5.30 mm to (87.7, 54.8), turned to 0 degrees
- moved R9 5.25 mm to (87.6, 56.9), turned to 0 degrees
- moved C7 2.86 mm to (71.8, 65.1), turned to -90 degrees
- moved C8 1.88 mm to (71.9, 57.4), turned to 90 degrees
- moved TP6 1.73 mm to (59.2, 58.8)
Connections:
- J2 pad 1: +3.3V -> /ESP_TMS
- J2 pad 2: /ESP_TMS -> /ESP_TCK
- J2 pad 3: GND -> /ESP_TDO
- J2 pad 4: /ESP_TCK -> /ESP_TDI
Routing:
- net GND: track 107.7 -> 184.0 mm, vias 24 -> 27
- net /Alarm_OFF_FILTERED: track 0.00 -> 48.8 mm, vias 0 -> 2
- net /BUZZER_GPIO_OUT: track 0.00 -> 47.4 mm, vias 0 -> 2
- net +3.3V: track 87.2 -> 112.4 mm, vias 3 -> 8
- net /ESP_TMS: track 0.00 -> 21.5 mm, vias 0 -> 2
- net /ESP_TDI: track 0.00 -> 19.3 mm
- net /ESP_TDO: track 0.00 -> 17.1 mm
- net /ESP_TCK: track 0.00 -> 15.7 mm
- net +5V: track 11.1 -> 20.7 mm
- net /ESP_IO0: track 53.1 -> 60.3 mm
- net /OE: track 45.9 -> 39.3 mm
- net /CS_MAX7221: track 30.8 -> 34.2 mm
- net Net-(D2-Pad+): track 0.00 -> 2.18 mm
- net /MOSI_MAX7221: track 31.3 -> 33.3 mm
- net /LFLAG: track 35.2 -> 36.1 mm
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