File: Hardware_design/Hardware_design.kicad_pcb (KiCad board)
At the start: 2 copper layers, 231.3 x 191.9 mm, 195 parts, among them IC1 ESP32-S3-WROOM-1-N16, J1 FTSH-103-01-F-D, J2 Conn_01x04_Pin, J3 54-00131, Q1 MMBT2222A, SW1 TL3301FF160QG, SW10 ADTS24NV, SW11 ADTS24NV, SW2 TL3301FF160QG, SW3 ADTS24NV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

Commit message: almost finished
just missing final conections and verification of constrains for fabrication
Parts:
- J2: footprint Footprints:Jtag_pins -> Footprints:4_pin_FTR-104-01-L-S
- moved C28 20.7 mm to (237.8, 192.8)
- moved R26 20.7 mm to (241.7, 191.2)
- moved R31 20.7 mm to (241.6, 193.9)
- moved TP15 4.26 mm to (227.6, 151.8)
- moved C5 3.51 mm to (68.4, 66.1)
- moved J2 2.94 mm to (77.4, 52.1)
- moved R11 1.98 mm to (84.4, 68.7)
- moved TP1 1.98 mm to (85.4, 71.9)
- moved C13 1.98 mm to (77.2, 58.4)
- moved D2 1.98 mm to (87.7, 56.8)
- moved R9 1.98 mm to (87.6, 58.9)
- moved TP2 1.98 mm to (81.5, 57.4)
- moved U3 1.98 mm to (81.2, 63.2)
- moved C12 1.97 mm to (90.0, 66.0)
- moved C37 1.97 mm to (93.5, 66.0)
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Routing:
- net /Display_management/SEG_F_MAX7221_8: track 0.00 -> 211.0 mm, vias 0 -> 2
- net /Display_management/SEG_D_MAX7221_8: track 0.00 -> 206.8 mm
- net /Display_management/SEG_B_MAX7221_8: track 0.00 -> 205.3 mm, vias 0 -> 4
- net /Display_management/SEG_F_MAX7221_4: track 0.00 -> 203.2 mm, vias 0 -> 2
- net /Display_management/SEG_A_MAX7221_8: track 0.00 -> 202.4 mm, vias 0 -> 10
- net /Display_management/SEG_C_MAX7221_8: track 0.00 -> 199.1 mm, vias 0 -> 10
- net /Display_management/SEG_DP_MAX7221_8: track 0.00 -> 198.0 mm, vias 0 -> 4
- net /Display_management/SEG_B_MAX7221_4: track 0.00 -> 192.8 mm, vias 0 -> 8
- net /Display_management/SEG_A_MAX7221_4: track 0.00 -> 192.2 mm, vias 0 -> 10
- net /Display_management/SEG_E_MAX7221_8: track 0.00 -> 191.0 mm, vias 0 -> 8
- net /Display_management/SEG_G_MAX7221_8: track 0.00 -> 188.3 mm, vias 0 -> 10
- net Net-(U11-DOUT): track 0.00 -> 184.4 mm, vias 0 -> 2
- net /Display_management/SEG_D_MAX7221_4: track 0.00 -> 178.8 mm
- net /Display_management/SEG_G_MAX7221_4: track 0.00 -> 175.6 mm, vias 0 -> 10
- net /Display_management/DIG_7_MAX7221_8: track 0.00 -> 173.0 mm, vias 0 -> 2
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