File: Hardware_design/Hardware_design.kicad_pcb (KiCad board)
At the start: 2 copper layers, 231.3 x 191.9 mm, 195 parts, among them IC1 ESP32-S3-WROOM-1-N16, J1 FTSH-103-01-F-D, J2 Conn_01x04_Pin, J3 54-00131, Q1 MMBT2222A, SW1 TL3301FF160QG, SW10 ADTS24NV, SW11 ADTS24NV, SW2 TL3301FF160QG, SW3 ADTS24NV, SW4 ADTS24NV, SW5 ADTS24NV, SW6 ADTS24NV, SW7 ADTS24NV, SW8 ADTS24NV, SW9 ADTS24NV, U1 LS7366R-S, U10 MAX7221CWG_, U11 MAX7221CWG_, U12 MAX7221CWG_, U15 74HC14D_653, U16 74HC14D_653, U2 TXB0104DR, U3 LP3875EMP-3.3, U4 MAX7221CWG_, U5 MAX7221CWG_, U6 MAX7221CWG_, U7 MAX7221CWG_, U8 MAX7221CWG_, U9 MAX7221CWG_

Commit message: almost finished
all conections made, need to fixed errors and warnings, minimum via size error for hole and diameter, also silkscreen text error.
Parts:
- moved E1 12.1 mm to (51.0, 75.8)
- moved TP4 7.31 mm to (59.4, 77.4)
- moved TP8 4.01 mm to (97.4, 48.9)
- moved C9 3.80 mm to (79.8, 39.2)
- moved C35 3.09 mm to (83.1, 37.5)
- moved C10 2.33 mm to (86.9, 36.4), turned to 90 degrees
- moved TP3 1.72 mm to (90.0, 69.5)
- moved C14 0.60 mm to (102.8, 33.3)
- moved R12 0.60 mm to (108.7, 33.0)
- moved U4 0.60 mm to (101.4, 32.9)
Connections:
- DS1 pad 3: /Display_management/DIG_0_MAX7221_1 -> unconnected-(DS1-COM_K_1-Pad3)
- DS10 pad 8: /Display_management/DIG_1_MAX7221_3 -> unconnected-(DS10-COM_K_2-Pad8)
- DS11 pad 3: /Display_management/DIG_2_MAX7221_3 -> unconnected-(DS11-COM_K_1-Pad3)
- DS12 pad 8: /Display_management/DIG_3_MAX7221_3 -> unconnected-(DS12-COM_K_2-Pad8)
- DS13 pad 3: /Display_management/DIG_0_MAX7221_4 -> unconnected-(DS13-COM_K_1-Pad3)
- DS14 pad 8: /Display_management/DIG_1_MAX7221_4 -> unconnected-(DS14-COM_K_2-Pad8)
- DS15 pad 3: /Display_management/DIG_2_MAX7221_4 -> unconnected-(DS15-COM_K_1-Pad3)
- DS16 pad 3: /Display_management/DIG_3_MAX7221_4 -> unconnected-(DS16-COM_K_1-Pad3)
- DS17 pad 3: /Display_management/DIG_0_MAX7221_5 -> unconnected-(DS17-COM_K_1-Pad3)
- DS18 pad 8: /Display_management/DIG_1_MAX7221_5 -> unconnected-(DS18-COM_K_2-Pad8)
- DS19 pad 3: /Display_management/DIG_2_MAX7221_5 -> unconnected-(DS19-COM_K_1-Pad3)
- DS2 pad 8: /Display_management/DIG_1_MAX7221_1 -> unconnected-(DS2-COM_K_2-Pad8)
- DS20 pad 8: /Display_management/DIG_3_MAX7221_5 -> unconnected-(DS20-COM_K_2-Pad8)
- DS21 pad 3: /Display_management/DIG_0_MAX7221_6 -> unconnected-(DS21-COM_K_1-Pad3)
- DS22 pad 8: /Display_management/DIG_1_MAX7221_6 -> unconnected-(DS22-COM_K_2-Pad8)
- DS23 pad 3: /Display_management/DIG_2_MAX7221_6 -> unconnected-(DS23-COM_K_1-Pad3)
- DS24 pad 3: /Display_management/DIG_3_MAX7221_6 -> unconnected-(DS24-COM_K_1-Pad3)
- DS25 pad 3: /Display_management/DIG_0_MAX7221_7 -> unconnected-(DS25-COM_K_1-Pad3)
- DS26 pad 8: /Display_management/DIG_1_MAX7221_7 -> unconnected-(DS26-COM_K_2-Pad8)
- DS27 pad 3: /Display_management/DIG_2_MAX7221_7 -> unconnected-(DS27-COM_K_1-Pad3)
- DS28 pad 8: /Display_management/DIG_3_MAX7221_7 -> unconnected-(DS28-COM_K_2-Pad8)
- DS29 pad 3: /Display_management/DIG_0_MAX7221_8 -> unconnected-(DS29-COM_K_1-Pad3)
- DS3 pad 3: /Display_management/DIG_2_MAX7221_1 -> unconnected-(DS3-COM_K_1-Pad3)
- DS30 pad 8: /Display_management/DIG_1_MAX7221_8 -> unconnected-(DS30-COM_K_2-Pad8)
- DS31 pad 3: /Display_management/DIG_2_MAX7221_8 -> unconnected-(DS31-COM_K_1-Pad3)
- DS32 pad 3: /Display_management/DIG_3_MAX7221_8 -> unconnected-(DS32-COM_K_1-Pad3)
- DS33 pad 8: /Display_management/DIG_0_MAX7221_9 -> unconnected-(DS33-COM_K_2-Pad8)
- DS34 pad 8: /Display_management/DIG_1_MAX7221_9 -> unconnected-(DS34-COM_K_2-Pad8)
- DS35 pad 8: /Display_management/DIG_2_MAX7221_9 -> unconnected-(DS35-COM_K_2-Pad8)
- DS36 pad 8: /Display_management/DIG_3_MAX7221_9 -> unconnected-(DS36-COM_K_2-Pad8)
- DS4 pad 8: /Display_management/DIG_3_MAX7221_1 -> unconnected-(DS4-COM_K_2-Pad8)
- DS45 pad 3: /Display_management/DIG_4_MAX7221_1 -> unconnected-(DS45-COM_K_1-Pad3)
- DS46 pad 8: /Display_management/DIG_5_MAX7221_1 -> unconnected-(DS46-COM_K_2-Pad8)
- DS47 pad 3: /Display_management/DIG_6_MAX7221_1 -> unconnected-(DS47-COM_K_1-Pad3)
- DS48 pad 8: /Display_management/DIG_7_MAX7221_1 -> unconnected-(DS48-COM_K_2-Pad8)
- DS49 pad 3: /Display_management/DIG_4_MAX7221_2 -> unconnected-(DS49-COM_K_1-Pad3)
- DS5 pad 3: /Display_management/DIG_0_MAX7221_2 -> unconnected-(DS5-COM_K_1-Pad3)
- DS50 pad 8: /Display_management/DIG_5_MAX7221_2 -> unconnected-(DS50-COM_K_2-Pad8)
- DS51 pad 8: /Display_management/DIG_6_MAX7221_2 -> unconnected-(DS51-COM_K_2-Pad8)
- DS52 pad 8: /Display_management/DIG_7_MAX7221_2 -> unconnected-(DS52-COM_K_2-Pad8)
- DS53 pad 3: /Display_management/DIG_4_MAX7221_3 -> unconnected-(DS53-COM_K_1-Pad3)
- DS54 pad 8: /Display_management/DIG_5_MAX7221_3 -> unconnected-(DS54-COM_K_2-Pad8)
- DS55 pad 3: /Display_management/DIG_6_MAX7221_3 -> unconnected-(DS55-COM_K_1-Pad3)
- DS56 pad 8: /Display_management/DIG_7_MAX7221_3 -> unconnected-(DS56-COM_K_2-Pad8)
- DS57 pad 3: /Display_management/DIG_4_MAX7221_4 -> unconnected-(DS57-COM_K_1-Pad3)
- DS58 pad 8: /Display_management/DIG_5_MAX7221_4 -> unconnected-(DS58-COM_K_2-Pad8)
- DS59 pad 8: /Display_management/DIG_6_MAX7221_4 -> unconnected-(DS59-COM_K_2-Pad8)
- DS6 pad 8: /Display_management/DIG_1_MAX7221_2 -> unconnected-(DS6-COM_K_2-Pad8)
- DS60 pad 8: /Display_management/DIG_7_MAX7221_4 -> unconnected-(DS60-COM_K_2-Pad8)
- DS61 pad 3: /Display_management/DIG_4_MAX7221_5 -> unconnected-(DS61-COM_K_1-Pad3)
- DS62 pad 8: /Display_management/DIG_5_MAX7221_5 -> unconnected-(DS62-COM_K_2-Pad8)
- DS63 pad 3: /Display_management/DIG_6_MAX7221_5 -> unconnected-(DS63-COM_K_1-Pad3)
- DS64 pad 8: /Display_management/DIG_7_MAX7221_5 -> unconnected-(DS64-COM_K_2-Pad8)
- DS65 pad 3: /Display_management/DIG_4_MAX7221_6 -> unconnected-(DS65-COM_K_1-Pad3)
- DS66 pad 8: /Display_management/DIG_5_MAX7221_6 -> unconnected-(DS66-COM_K_2-Pad8)
- DS67 pad 8: /Display_management/DIG_6_MAX7221_6 -> unconnected-(DS67-COM_K_2-Pad8)
- DS68 pad 8: /Display_management/DIG_7_MAX7221_6 -> unconnected-(DS68-COM_K_2-Pad8)
- DS69 pad 3: /Display_management/DIG_4_MAX7221_7 -> unconnected-(DS69-COM_K_1-Pad3)
- DS7 pad 3: /Display_management/DIG_2_MAX7221_2 -> unconnected-(DS7-COM_K_1-Pad3)
- DS70 pad 8: /Display_management/DIG_5_MAX7221_7 -> unconnected-(DS70-COM_K_2-Pad8)
- DS71 pad 3: /Display_management/DIG_6_MAX7221_7 -> unconnected-(DS71-COM_K_1-Pad3)
- DS72 pad 8: /Display_management/DIG_7_MAX7221_7 -> unconnected-(DS72-COM_K_2-Pad8)
- DS73 pad 3: /Display_management/DIG_4_MAX7221_8 -> unconnected-(DS73-COM_K_1-Pad3)
- DS74 pad 8: /Display_management/DIG_5_MAX7221_8 -> unconnected-(DS74-COM_K_2-Pad8)
- DS75 pad 8: /Display_management/DIG_6_MAX7221_8 -> unconnected-(DS75-COM_K_2-Pad8)
- DS76 pad 8: /Display_management/DIG_7_MAX7221_8 -> unconnected-(DS76-COM_K_2-Pad8)
- DS8 pad 8: /Display_management/DIG_3_MAX7221_2 -> unconnected-(DS8-COM_K_2-Pad8)
- DS9 pad 3: /Display_management/DIG_0_MAX7221_3 -> unconnected-(DS9-COM_K_1-Pad3)
Routing:
- net /SCK_MAX7221_5V: track 165.2 -> 401.1 mm, vias 0 -> 16
- net /CS_MAX7221_5V: track 178.0 -> 376.7 mm, vias 4 -> 18
- net +5V: track 27.4 -> 213.6 mm, vias 0 -> 6
- net /Display_management/SEG_B_MAX7221_6: track 116.6 -> 203.8 mm
- net /Display_management/SEG_A_MAX7221_6: track 114.4 -> 201.0 mm
- net /Display_management/SEG_E_MAX7221_6: track 103.8 -> 187.4 mm
- net GND: track 184.8 -> 268.3 mm, vias 26 -> 66
- net /Display_management/SEG_C_MAX7221_6: track 116.0 -> 199.1 mm
- net /Display_management/SEG_D_MAX7221_6: track 121.0 -> 203.9 mm
- net /Display_management/SEG_DP_MAX7221_6: track 115.5 -> 198.3 mm
- net /Display_management/SEG_F_MAX7221_6: track 128.9 -> 211.5 mm
- net /Display_management/SEG_G_MAX7221_6: track 106.5 -> 188.5 mm
- net /Display_management/DIG_7_MAX7221_6: track 102.8 -> 177.1 mm, vias 1 -> 2
- net /Display_management/DIG_6_MAX7221_6: track 102.2 -> 151.5 mm, vias 1 -> 2
- net /Display_management/DIG_7_MAX7221_4: track 102.8 -> 149.5 mm, vias 1 -> 2
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
Commit message: final design
Parts:
- added REF**: MountingHole_2.5mm, MountingHole:MountingHole_2.5mm, F.Cu at (42.3, 31.2)
- added REF**: MountingHole_2.5mm, MountingHole:MountingHole_2.5mm, F.Cu at (260.8, 202.6)
- added REF**: MountingHole_2.5mm, MountingHole:MountingHole_2.5mm, F.Cu at (46.4, 92.4)
- added REF**: MountingHole_2.5mm, MountingHole:MountingHole_2.5mm, F.Cu at (263.6, 24.1)
- added REF**: MountingHole_2.5mm, MountingHole:MountingHole_2.5mm, F.Cu at (96.6, 203.6)
- C1, C2, C3, C7: value 0.1uF -> 0.1 uF
- C11: footprint Footprints:0805_SMD_CERAMIC_CAP_T491B106K016AT -> Footprints:CAP_0603_CAPC1608X90N
- C14, C15, C16, C17, C18, C19, C20, C21, C22: moved to B.Cu
- moved J3 2.85 mm to (46.5, 102.0)
- moved C15 1.98 mm to (107.6, 57.8)
- moved C22 1.98 mm to (235.6, 159.4)
- moved C20 1.12 mm to (103.4, 172.2)
- moved C14 0.58 mm to (102.2, 33.2)
- moved TP8 0.58 mm to (96.8, 48.9)
- moved C11 0.31 mm to (44.8, 37.5)
- moved C29 0.13 mm to (64.1, 94.1)
- moved C16 0.10 mm to (103.0, 79.5)
Routing:
- net +5V: track 213.6 -> 234.7 mm, vias 6 -> 13
- net GND: track 268.3 -> 248.4 mm, vias 66 -> 58
- net /Display_management/DIG_3_MAX7221_1: track 66.1 -> 73.5 mm
- net +3.3V: vias 8 -> 7
