File: Hardware_design/Hardware_design.kicad_pcb (KiCad board)
At the start: 2 copper layers, 231.3 x 191.9 mm, 200 parts, among them IC1 ESP32-S3-WROOM-1-N16, J1 FTSH-103-01-F-D, J2 Conn_01x04_Pin, J3 54-00131, Q1 MMBT2222A, SW1 TL3301FF160QG, SW10 ADTS24NV, SW11 ADTS24NV, SW2 TL3301FF160QG, SW3 ADTS24NV, SW4 ADTS24NV, SW5 ADTS24NV, SW6 ADTS24NV, SW7 ADTS24NV, SW8 ADTS24NV, SW9 ADTS24NV, U1 LS7366R-S, U10 MAX7221CWG_, U11 MAX7221CWG_, U12 MAX7221CWG_, U15 74HC14D_653, U16 74HC14D_653, U2 TXB0104DR, U3 LP3875EMP-3.3, U4 MAX7221CWG_, U5 MAX7221CWG_, U6 MAX7221CWG_, U7 MAX7221CWG_, U8 MAX7221CWG_, U9 MAX7221CWG_

Commit message: first working attempt
Parts:
- moved Q1 0.19 mm to (89.2, 88.2)
Changed lines of the file:
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@@
 	(generator_version "10.0")
 	(general
-		(thickness 1.6)
+		(thickness 1.69)
 		(legacy_teardrops no)
 	)
@@
 			(layer "dielectric 1"
 				(type "core")
-				(thickness 1.51)
+				(thickness 1.6)
 				(material "FR4")
 				(epsilon_r 4.5)
@@
 		(capping no)
 		(filling no)
+		(zone_defaults)
 		(pcbplotparams
 			(layerselection 0x00000000_00000000_55555555_5755f5df)
@@
 	(footprint "Footprints:TRANSISTOR_MMBT2222A"
 		(layer "F.Cu")
-		(at 88.96 88.21 90)
+		(at 89.15 88.21 90)
 		(property "Reference" "Q1"
-			(at 2.785 1.015 180)
+			(at 2.77 1.21 180)
 			(layer "F.SilkS")
 			(effects
@@
 			)
 		)
-		(property "PARTREV" "2024-03-11"
-			(at 0 0 90)
-			(unlocked yes)
-			(layer "F.Fab")
-			(hide yes)
-			(effects
-				(font
-					(size 1 1)
-					(thickness 0.15)
-				)
-			)
-		)
-		(property "STANDARD" "IPC 7351B"
-			(at 0 0 90)
-			(unlocked yes)
-			(layer "F.Fab")
-			(hide yes)
-			(effects
-				(font
-					(size 1 1)
-					(thickness 0.15)
-				)
-			)
-		)
-		(property "SNAPEDA_PACKAGE_ID" "124619"
-			(at 0 0 90)
-			(unlocked yes)
-			(layer "F.Fab")
-			(hide yes)
-			(effects
-				(font
-					(size 1 1)
-					(thickness 0.15)
-				)
-			)
-		)
-		(property "MAXIMUM_PACKAGE_HEIGHT" "1.20mm"
-			(at 0 0 90)
-			(unlocked yes)
-			(layer "F.Fab")
-			(hide yes)
-			(effects
-				(font
-					(size 1 1)
-					(thickness 0.15)
-				)
-			)
-		)
-		(property "MANUFACTURER" "Diotec"
-			(at 0 0 90)
-			(unlocked yes)
-			(layer "F.Fab")
-			(hide yes)
-			(effects
-				(font
-					(size 1 1)
-					(thickness 0.15)
-				)
-			)
-		)
 		(sheetname "/")
 		(sheetfile "Hardware_design.kicad_sch")
-		(units
-			(unit
-				(name "A")
-				(pins "1" "3" "2")
-			)
-		)
 		(attr smd)
 		(duplicate_pad_numbers_are_jumpers no)
@@
 		)
 		(pad "1" smd roundrect
-			(at -1 -0.95 90)
+			(at -1 -1.025 90)
 			(size 1.32 0.6)
 			(layers "F.Cu" "F.Mask" "F.Paste")
@@
 		)
 		(pad "2" smd roundrect
-			(at -1 0.95 90)
+			(at -1 1.025 90)
 			(size 1.32 0.6)
 			(layers "F.Cu" "F.Mask" "F.Paste")
@@
 		(at 44.79 37.51 180)
 		(property "Reference" "C11"
-			(at 0.432 -1.2064 0)
+			(at 2.38 -0.7 0)
 			(layer "F.SilkS")
 			(effects
@@
 	)
 	(segment
-		(start 43.7225 37.505)
-		(end 41.455 37.505)
-		(width 0.508)
+		(start 48.64 32.63)
+		(end 48.11 32.1)
+		(width 0.762)
 		(layer "F.Cu")
 		(net "GND")
 	)
 	(segment
-		(start 48.64 32.63)
-		(end 48.11 32.1)
-		(width 0.762)
+		(start 41.63 36.19)
+		(end 42.945 37.505)
+		(width 0.508)
 		(layer "F.Cu")
 		(net "GND")
@@
 	)
 	(segment
-		(start 96.77 174.075)
-		(end 98.05 174.075)
+		(start 42.945 37.505)
+		(end 43.7225 37.505)
 		(width 0.508)
 		(layer "F.Cu")
@@
 	)
 	(segment
-		(start 69.205 74.23)
-		(end 71.605 74.23)
+		(start 96.77 174.075)
+		(end 98.05 174.075)
 		(width 0.508)
 		(layer "F.Cu")
@@
 	)
 	(segment
-		(start 41.455 37.505)
-		(end 41.36 37.41)
+		(start 69.205 74.23)
+		(end 71.605 74.23)
 		(width 0.508)
 		(layer "F.Cu")
@@
 	)
 	(via
-		(at 41.36 37.41)
+		(at 41.63 36.19)
 		(size 1.016)
 		(drill 0.508)
@@
 	)
 	(segment
-		(start 89.91 93.85)
-		(end 89.94 93.88)
+		(start 90.18 89.275)
+		(end 90.18 93.64)
 		(width 0.762)
 		(layer "F.Cu")
@@
 	)
 	(segment
-		(start 89.91 89.21)
-		(end 89.91 93.85)
+		(start 90.18 93.64)
+		(end 89.94 93.88)
 		(width 0.762)
 		(layer "F.Cu")
