File: Hardware_design/Display_management.kicad_sch (KiCad schematic)
At the start: 97 parts, among them U10 MAX7221CWG_, U11 MAX7221CWG_, U12 MAX7221CWG_, U4 MAX7221CWG_, U5 MAX7221CWG_, U6 MAX7221CWG_, U7 MAX7221CWG_, U8 MAX7221CWG_, U9 MAX7221CWG_

Commit message: almost finished
all conections made, need to fixed errors and warnings, minimum via size error for hole and diameter, also silkscreen text error.
Connections:
- net DIG_0_MAX7221_1: no longer DS1.3 (COM_K_1)
- net DIG_0_MAX7221_2: no longer DS5.3 (COM_K_1)
- net DIG_0_MAX7221_3: no longer DS9.3 (COM_K_1)
- net DIG_0_MAX7221_4: no longer DS13.3 (COM_K_1)
- net DIG_0_MAX7221_5: no longer DS17.3 (COM_K_1)
- net DIG_0_MAX7221_6: no longer DS21.3 (COM_K_1)
- net DIG_0_MAX7221_7: no longer DS25.3 (COM_K_1)
- net DIG_0_MAX7221_8: no longer DS29.3 (COM_K_1)
- net DIG_0_MAX7221_9: no longer DS33.8 (COM_K_2)
- net DIG_1_MAX7221_1: no longer DS2.8 (COM_K_2)
- net DIG_1_MAX7221_2: no longer DS6.8 (COM_K_2)
- net DIG_1_MAX7221_3: no longer DS10.8 (COM_K_2)
- net DIG_1_MAX7221_4: no longer DS14.8 (COM_K_2)
- net DIG_1_MAX7221_5: no longer DS18.8 (COM_K_2)
- net DIG_1_MAX7221_6: no longer DS22.8 (COM_K_2)
- net DIG_1_MAX7221_7: no longer DS26.8 (COM_K_2)
- net DIG_1_MAX7221_8: no longer DS30.8 (COM_K_2)
- net DIG_1_MAX7221_9: no longer DS34.8 (COM_K_2)
- net DIG_2_MAX7221_1: no longer DS3.3 (COM_K_1)
- net DIG_2_MAX7221_2: no longer DS7.3 (COM_K_1)
- net DIG_2_MAX7221_3: no longer DS11.3 (COM_K_1)
- net DIG_2_MAX7221_4: no longer DS15.3 (COM_K_1)
- net DIG_2_MAX7221_5: no longer DS19.3 (COM_K_1)
- net DIG_2_MAX7221_6: no longer DS23.3 (COM_K_1)
- net DIG_2_MAX7221_7: no longer DS27.3 (COM_K_1)
- net DIG_2_MAX7221_8: no longer DS31.3 (COM_K_1)
- net DIG_2_MAX7221_9: no longer DS35.8 (COM_K_2)
- net DIG_3_MAX7221_1: no longer DS4.8 (COM_K_2)
- net DIG_3_MAX7221_2: no longer DS8.8 (COM_K_2)
- net DIG_3_MAX7221_3: no longer DS12.8 (COM_K_2)
- net DIG_3_MAX7221_4: no longer DS16.3 (COM_K_1)
- net DIG_3_MAX7221_5: no longer DS20.8 (COM_K_2)
- net DIG_3_MAX7221_6: no longer DS24.3 (COM_K_1)
- net DIG_3_MAX7221_7: no longer DS28.8 (COM_K_2)
- net DIG_3_MAX7221_8: no longer DS32.3 (COM_K_1)
- net DIG_3_MAX7221_9: no longer DS36.8 (COM_K_2)
- net DIG_4_MAX7221_1: no longer DS45.3 (COM_K_1)
- net DIG_4_MAX7221_2: no longer DS49.3 (COM_K_1)
- net DIG_4_MAX7221_3: no longer DS53.3 (COM_K_1)
- net DIG_4_MAX7221_4: no longer DS57.3 (COM_K_1)
- net DIG_4_MAX7221_5: no longer DS61.3 (COM_K_1)
- net DIG_4_MAX7221_6: no longer DS65.3 (COM_K_1)
- net DIG_4_MAX7221_7: no longer DS69.3 (COM_K_1)
- net DIG_4_MAX7221_8: no longer DS73.3 (COM_K_1)
- net DIG_5_MAX7221_1: no longer DS46.8 (COM_K_2)
- net DIG_5_MAX7221_2: no longer DS50.8 (COM_K_2)
- net DIG_5_MAX7221_3: no longer DS54.8 (COM_K_2)
- net DIG_5_MAX7221_4: no longer DS58.8 (COM_K_2)
- net DIG_5_MAX7221_5: no longer DS62.8 (COM_K_2)
- net DIG_5_MAX7221_6: no longer DS66.8 (COM_K_2)
- net DIG_5_MAX7221_7: no longer DS70.8 (COM_K_2)
- net DIG_5_MAX7221_8: no longer DS74.8 (COM_K_2)
- net DIG_6_MAX7221_1: no longer DS47.3 (COM_K_1)
- net DIG_6_MAX7221_2: no longer DS51.8 (COM_K_2)
- net DIG_6_MAX7221_3: no longer DS55.3 (COM_K_1)
- net DIG_6_MAX7221_4: no longer DS59.8 (COM_K_2)
- net DIG_6_MAX7221_5: no longer DS63.3 (COM_K_1)
- net DIG_6_MAX7221_6: no longer DS67.8 (COM_K_2)
- net DIG_6_MAX7221_7: no longer DS71.3 (COM_K_1)
- net DIG_6_MAX7221_8: no longer DS75.8 (COM_K_2)
- net DIG_7_MAX7221_1: no longer DS48.8 (COM_K_2)
- net DIG_7_MAX7221_2: no longer DS52.8 (COM_K_2)
- net DIG_7_MAX7221_3: no longer DS56.8 (COM_K_2)
- net DIG_7_MAX7221_4: no longer DS60.8 (COM_K_2)
- net DIG_7_MAX7221_5: no longer DS64.8 (COM_K_2)
- net DIG_7_MAX7221_6: no longer DS68.8 (COM_K_2)
- net DIG_7_MAX7221_7: no longer DS72.8 (COM_K_2)
- net DIG_7_MAX7221_8: no longer DS76.8 (COM_K_2)
- no-connect marks 5 -> 73
