File: Hardware_design/Hardware_design.kicad_sch (KiCad schematic)
At the start: 50 parts, among them IC1 ESP32-S3-WROOM-1-N16, J1 FTSH-103-01-F-D, J2 Conn_01x04_Pin, J3 54-00131, Q1 MMBT2222A, SW1 TL3301FF160QG, SW2 TL3301FF160QG, U1 LS7366R-S, U2 TXB0104DR, U3 LP3875EMP-3.3

Commit message: final design
Parts:
- C1, C2, C3, C7: value 0.1uF -> 0.1 uF
- C11: footprint Footprints:0805_SMD_CERAMIC_CAP_T491B106K016AT -> Footprints:CAP_0603_CAPC1608X90N
Changed lines of the file:
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@@
 			)
 		)
-		(property "Footprint" "Footprints:0805_SMD_CERAMIC_CAP_T491B106K016AT"
+		(property "Footprint" "Footprints:CAP_0603_CAPC1608X90N"
 			(at 202.2348 50.8 0)
 			(hide yes)
@@
 			)
 		)
-		(property "Value" "0.1uF"
+		(property "Value" "0.1 uF"
 			(at 144.272 65.024 0)
 			(show_name no)
@@
 			)
 		)
-		(property "Value" "0.1uF"
+		(property "Value" "0.1 uF"
 			(at 332.74 105.4099 90)
 			(show_name no)
@@
 			)
 		)
-		(property "Value" "0.1uF"
+		(property "Value" "0.1 uF"
 			(at 374.65 104.1399 90)
 			(show_name no)
@@
 			)
 		)
-		(property "Value" "0.1uF"
+		(property "Value" "0.1 uF"
 			(at 226.568 51.054 0)
 			(show_name no)
